File: Theremin.kicad_sch (KiCad schematic)
At the start: 32 parts, among them Q1 2N5458, Q2 2N5458, Q3 2N5458, U1 LM7806_TO220

Commit message: PCB y esquemático posiblemente finalizado
Parts:
- removed AE1: Antenna, symbol Device:Antenna
- added J1, J2: Conn_01x02_Pin, Connector_Wire:SolderWire-0.1sqmm_1x02_P3.6mm_D0.4mm_OD1mm, symbol Connector:Conn_01x02_Pin
- added J3: Antenna Conn_01x01_Pin, Connector_Wire:SolderWire-0.1sqmm_1x01_D0.4mm_OD1mm, symbol Connector:Conn_01x01_Pin
- C1, C11, C12, C2, C3, C9: footprint Capacitor_THT:CP_Radial_D5.0mm_P2.00mm -> Capacitor_THT:CP_Radial_D4.0mm_P1.50mm
- C10: footprint Capacitor_THT:C_Rect_L4.0mm_W2.5mm_P2.50mm -> Capacitor_THT:C_Rect_L4.6mm_W2.0mm_P2.50mm_MKS02_FKP02
- C15, C7: footprint (none) -> Capacitor_THT:C_Disc_D3.0mm_W1.6mm_P2.50mm
- C6: footprint Capacitor_SMD:C_Trimmer_Murata_TZB4-A -> Capacitor_THT:CP_Radial_D4.0mm_P1.50mm
- L1, L2: footprint Transistor_THT:L_Axial_L6.6mm_D2.7mm_P10.16mm_Horizontal_Vishay_IM-2 -> Transistor_THT:L_Axial_L5.3mm_D2.2mm_P10.16mm_Horizontal_Vishay_IM-1
- Q1, Q2, Q3: footprint Package_TO_SOT_THT:TO-92 -> Package_TO_SOT_THT:TO-92_Inline
- R1, R9: footprint Resistor_THT:R_Axial_DIN0207_L6.3mm_D2.5mm_P7.62mm_Horizontal -> Resistor_THT:R_Axial_DIN0204_L3.6mm_D1.6mm_P7.62mm_Horizontal
- R2, R4, R6, R8: footprint Resistor_THT:R_Axial_DIN0204_L3.6mm_D1.6mm_P5.08mm_Horizontal -> Resistor_THT:R_Axial_DIN0204_L3.6mm_D1.6mm_P7.62mm_Horizontal
- R3, R5, R7: footprint (none) -> Resistor_THT:R_Axial_DIN0204_L3.6mm_D1.6mm_P7.62mm_Horizontal
Connections:
- net +9V: now also J2.1 (Pin_1)
- net GND: now also Q1.3 (G), Q3.3 (G), J1.2 (Pin_2), J2.2 (Pin_2); no longer Q1.2 (G), Q3.2 (G)
- net at C15.1, C7.2, R3.1: now also Q2.3 (G); no longer Q2.2 (G)
- net at C13.1, C15.2, L2.2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: now also J3.1 (Pin_1)
- net at C9.1, R4.1: now also Q2.2 (S); no longer Q2.3 (S)
- net at C13.2, C14.1, R8.1: now also Q3.2 (S); no longer Q3.3 (S)
- net at C4.2, C5.1, R2.1: now also Q1.2 (S); no longer Q1.3 (S)
- net at C10.1, R6.2, R7.1: now also J1.1 (Pin_1)
Other:
- note added: "9 volt battery input"
- note added: "Audio output"
